File: pcb/ppm2spi.sch (KiCad schematic (older format))
At the start: 46 parts, among them IC1 ATMEGA328-A, K1 CONN_3, P1 CONN_5, P2 CONN_6, P3 CONN_3X2, P4 CONN_9, P5 CONN_2, P6 CONN_4, P7 CONN_2, SW1 SW_PUSH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

Commit message: Update of schematic comments to reflect new Spektrum channel order option. Also MOSI is now floating during read in's. This makes for nicer treatment of the A7105.
Other:
- note added: "JP2 shorting this link enables\nSpektrum channel order TAER.\nLink open gives Futaba channel order AETR."
- note removed: "JP2 enables alternative channel order\nAllows this module to work\nwith other transmitters\nCurrently unimplimented"
Changed lines of the file:
@@
-EESchema Schematic File Version 2  date 09/07/2013 21:25:35
+EESchema Schematic File Version 2
 LIBS:power
 LIBS:device
@@
 Sheet 1 1
 Title "ppm2spi Convertor"
-Date "9 jul 2013"
+Date "1 nov 2013"
 Rev "0.1"
 Comp "Copyright Cameron Weeks <th9xer@gmail.com>"
@@
 Alternative channel order\nCurrently unimplimented
 Text Notes 4600 5400 0    60   ~ 0
-JP2 enables alternative channel order\nAllows this module to work\nwith other transmitters\nCurrently unimplimented
+JP2 shorting this link enables\nSpektrum channel order TAER.\nLink open gives Futaba channel order AETR.
 Text Label 5000 3900 0    60   ~ 0
 Rx

Commit message: Updated comments on schematic
Other:
- note added: "Alternative channel order"
- note added: "Alternative channel order\nJP2 shorting this link enables\nSpektrum channel order TAER.\nLink open gives Futaba channel order AETR."
- note removed: "Alternative channel order\nCurrently unimplimented"
- note removed: "JP2 shorting this link enables\nSpektrum channel order TAER.\nLink open gives Futaba channel order AETR."
Changed lines of the file:
@@
 Sheet 1 1
 Title "ppm2spi Convertor"
-Date "1 nov 2013"
+Date "8 nov 2013"
 Rev "0.1"
 Comp "Copyright Cameron Weeks <th9xer@gmail.com>"
@@
 Bind
 Text Notes 6250 3300 0    60   ~ 0
-Alternative channel order\nCurrently unimplimented
+Alternative channel order
 Text Notes 4600 5400 0    60   ~ 0
-JP2 shorting this link enables\nSpektrum channel order TAER.\nLink open gives Futaba channel order AETR.
+Alternative channel order\nJP2 shorting this link enables\nSpektrum channel order TAER.\nLink open gives Futaba channel order AETR.
 Text Label 5000 3900 0    60   ~ 0
 Rx

Commit message: Changed 5v reg to a more common footprint, changed BOM to suit Updated schematic pdf Ready for the 2nd PCB batch I think.
Parts:
- U1: value XC6202P502PR -> MCP1703AT-5002E/MB
Changed lines of the file:
@@
 Comp "Copyright Cameron Weeks <th9xer@gmail.com>"
 Comment1 "Licensed under the TAPR Open Hardware License (www.tapr.org/OHL)"
-Comment2 ""
+Comment2 "http://code.google.com/p/rc-ppm-2-spi/"
 Comment3 ""
 Comment4 ""
@@
 P 8600 1600
 F 0 "U1" H 8750 1404 60  0000 C CNN
-F 1 "XC6202P502PR" H 8600 1800 60  0000 C CNN
+F 1 "MCP1703AT-5002E/MB" H 8600 1900 60  0000 C CNN
 F 2 "" H 8600 1600 60  0001 C CNN
 F 3 "" H 8600 1600 60  0001 C CNN
